File: _autosave-Transmi.kicad_pcb (KiCad board)
At the start: 2 copper layers, 232.6 x 140 mm, 344 parts, among them J101 Bat, J104 Ant, J105 Boot, Q101 Si2301CDS, Q102 XC6220B331MR-G, SW129 SK-3296S-01-L3, U1 ESP32-S2FH4, U103 TP4056, X101 S2240000101050JY, X102 Q13FC1350000400

Commit message: Expensive one
Parts:
- moved C166 9.57 mm to (71.0, 146.0), turned to -90 degrees
- moved H104 5.37 mm to (258.5, 152.2)
- moved H103 2.20 mm to (258.5, 22.5)
- moved H101 1.50 mm to (36.5, 23.0)
- moved H102 1.27 mm to (36.0, 152.5)
Routing:
- net Earth: track 1656.3 -> 1671.9 mm
- added copper zone on B.Cu, net VCC
